File: kicad/bebl_v2.sch (KiCad schematic (older format))
At the start: 36 parts, among them IC1 ATMEGA328, P14 I/O, P15 I/O, P16 I/O, P2 BAT, P6 LiPo, P7 GPS, P8 FTDI, P9 ISP, SW1 SW_PUSH, U1 3V3, X1 8MHz

Commit message: bebl_v2 work in progress
Parts:
- removed B1: AREF, ArthurC Lib:I%2fO, symbol I/O
- removed B10, B11: I/O, ArthurC Lib:I%2fO_ADR, symbol I/O
- removed B5, B6, B8, LED1, LED2, P14, P15, P16: I/O, ArthurC Lib:I%2fO, symbol I/O
- removed C2, C5: 1u, ArthurC Lib:c_0805, symbol C
- removed C3: 47uF_25V, ArthurC Lib:C_ELCO_SMD, symbol C_POL
- removed C7: 100n, ArthurC Lib:c_0805, symbol C
- removed D1, D2: LED, ArthurC Lib:d_0805, symbol LED
- removed P2: BAT, ArthurC Lib:pin_strip_2, symbol CONN_2
- removed P7: GPS, ArthurC Lib:PIN_ARRAY-9X1, symbol CONN_9
- removed R5, R8: 750E, ArthurC Lib:r_0805, symbol R
- removed U1: 3V3, ArthurC Lib:SOT23-3, symbol MCP_1700
- added C? (x2): 10uF, symbol C_POL
- added C? (x2): 4u7, symbol C_POL
- added C?: 100n, symbol C_NPOL
- added D? (x7): DIODE_LED, symbol DIODE_LED
- added L?: 4u7, symbol INDUCTOR
- added P?: USB-Micro, symbol USB-Micro
- added R?: 470, symbol R2
- added R?: 2k, symbol R2
- added R? (x6): R2, symbol R2
- added U?: TPS61221DCK, symbol TPS61221DCK
- added U?: MCP73831, SOT-23-5, symbol MCP73831
- renumbered P6 to P?
Connections:
- net labels added: Vusb
- net labels removed: 1pps, 3Vgps, A1, A2, A7, AREF, EN, FIX, GPS_BAT, GPS_Rx, GPS_Tx, Ir_Dat, LED1, LED2, PB0, PB1, SQW
- wire segments 113 -> 123
- no-connect marks 0 -> 3
Other:
- note added: "NOTES :\nKeep LiPo charger external to reduce complexity / cost.\nUse change over switch for LiPo Charge <> BEBL On"
- note removed: "External Battery\n3V Max."
- note removed: "External Battery\n9V Max."
- note removed: "GPS Header"
- note removed: "INDICATORS"
- note removed: "MCP1700T-3302E/TT"
- note removed: "VIN"
- moved on the sheet: P?

Commit message: bebl_v2 work in progress
Parts:
- removed D? (x6): DIODE_LED, symbol DIODE_LED
- removed PCB1: PCB, ArthurC Lib:PCB, symbol PCB
- removed R? (x6): R2, symbol R2
- added C? (x2): 100nF, c_0805, symbol C_NPOL
- added C?: 10uF, C_ELCO_SMD, symbol C_POL
- added D?: ZENER_2V7, symbol ZENER
- added P?: Alt_Add, ShortLink2, symbol CONN_3
- added P?: Int1, ShortLink2, symbol CONN_3
- added P?: Int2, ShortLink2, symbol CONN_3
- added P?: LED, symbol CONN_2
- added Q?: 2N5088BU, TO92-EBC, symbol NPN
- added Q?: MGSF1N03L, symbol MOSFET_N
- added R?: Rled, symbol R
- added R?: 22k, symbol R
- added SC? (x3): SCREW, ArthurC Lib:vite_3mm, symbol SCREW
- added U?: ADXL345, ADXL345, symbol ADXL345
- C1, C10, C11: symbol C -> C_NPOL
Connections:
- net +3.3V: now also C?.1, C?.1, C?.1, P?.1 (P1), P?.3 (P3), P?.3 (P3), P?.3 (P3), R?.1, U?.1 (VDD), U?.6 (VSS), U?.7 (CS)
- net GND: now also C?.2, C?.2, C?.2, D?.1 (A), P?.1 (P1), P?.1 (P1), P?.1 (P1), Q?.3 (E), R?.2, U?.2 (GND), U?.4 (GND1), U?.5 (GND2)
- net SCL: now also U?.14 (SCL)
- net SDA: now also U?.13 (SDA)
- net at IC1.32 (PD2(INT0)): now also D?.2 (K), Q?.2 (C), Q?.G, R?.2
- new net: Q?.1 (B), Q?.S, R?.1
- new net: P?.2 (PM), Q?.D
- new net ACL_INT1: P?.2 (P2), U?.8 (INT1)
- new net ACL_INT2: P?.2 (P2), U?.9 (INT2)
- new net ACL_SDO: P?.2 (P2), U?.12 (SDO)
- no-connect marks 3 -> 6
Other:
- note added: "Accelerometer, 3V3 I2C"
- note added: "Rled = 0.5/Iled\nW(Rled) = 0.25/Rled\n\n25Ohms for 20mA : 10mW\n\n6.25Ohm for 80mA : 40mW\n\n"
- moved on the sheet: R1, R2, SC1

Commit message: bebl_v2 work in progress
Parts:
- added B1, B10, B11, B12, B13, B2, B3, B4, B5, B6, B7, B8, B9: I/O, symbol I/O
- added D3: IND, symbol DIODE_LED
- added R8: 56E, symbol R
- D2: renamed from D?; value DIODE_LED -> CHG
- SW1: value SW_PUSH -> RST
- gave numbers to parts that had none: 28
- renumbered C10 to C1, C11 to C2, C1 to C3, P9 to P1, P8 to P2, R7 to R1, R1 to R2, R2 to R3, IC1 to U1
Connections:
- net GND: now also D3.2 (K)
- net SS: now also B13.1
- net at U1.1 (PD3(INT1)): now also B8.1
- net LED: now reaches U1.10 (PD6(AIN0))
- net LED: now also D1.2 (K), Q1.2 (C), Q2.G, R4.2
- net at U1.11 (PD7(AIN1)): now also B10.1
- net at U1.12 (PB0(ICP)): now also B11.1
- net at U1.13 (PB1(OC1A)): now also B12.1
- net at U1.19 (ADC6): now also B5.1
- net at U1.2 (PD4(XCK/T0)): now also B9.1
- net at U1.22 (ADC7): now also B6.1
- net at U1.23 (PC0(ADC0)): now also B1.1
- net at U1.24 (PC1(ADC1)): now also B2.1
- net at U1.25 (PC2(ADC2)): now also B3.1
- net at U1.26 (PC3(ADC3)): now also B4.1
- net at U1.9 (PD5(T1)): now also R8.2
- net L: now reaches L1.2, U4.5 (L)
- net PROG: now reaches R7.2, U3.5 (Prog)
- new net: B7.1, U1.32 (PD2(INT0))
- new net: D3.1 (A), R8.1
Other:
- note added: "1x LED 20mA, 5mm, 9000mcd\n(On Indicator, Drive Light DRL)"
- note added: "4x LED 80mA, 10mm, 12000mcd, (48000mcd, 320mA)\nor\n5x LED 20mA, 5mm, 9000mcd, (45000mcd, 100mA)"
- note added: "ACCELEROMETER, I2C"
- note added: "LED DRIVER"
- note added: "LiPo CHARGER"
- note added: "Rled = 0.5/Iled\nW(Rled) = 0.25/Rled\n5 Ohms for 100mA : 50mW\n1.56 Ohms for 320mA : 160mW\n\n"
- note added: "VOLTAGE REGULATOR"
- note removed: "Accelerometer, 3V3 I2C"
- note removed: "NOTES :\nKeep LiPo charger external to reduce complexity / cost.\nUse change over switch for LiPo Charge <> BEBL On"
- note removed: "Rled = 0.5/Iled\nW(Rled) = 0.25/Rled\n\n25Ohms for 20mA : 10mW\n\n6.25Ohm for 80mA : 40mW\n\n"
- moved on the sheet: C10, C11, C5, C6, C7, C8, C9, D1, D2, L1, P3, P4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
