File: kicad/bebl_v2.sch (KiCad schematic (older format))
At the start: 71 parts, among them P1 ISP, P10 LED_DRL, P11 DRV_LED, P12 CHG_LED, P13 LED_CHG, P2 FTDI, P3 Ext_LiPo, P4 USB-Micro, P8 DRL_LED, P9 LED_DRV, SW1 RST, SW2 MODE, U1 ATMEGA328, U3 ADXL345, U4 MCP73831, U5 TPS61221DCK, X1 8MHz

Commit message: modified schematic for transistor drive
Parts:
- removed D1: DRL, bebl_v2_pretty:LED-5MM, symbol DIODE_LED
- removed D2, D3, D4, D5, D6: LED_R, bebl_v2_pretty:LED-5MM, symbol DIODE_LED
- removed D8: CHG, bebl_v2_pretty:LED-0805, symbol DIODE_LED
- removed P13: LED_CHG, bebl_v2_pretty:pin_strip_2, symbol CONN_2
- removed Q? (x6): BC847BDW1T1G, SOT-363, symbol BC847BDW1T1G
- removed R? (x6): 56E, bebl_v2_pretty:r_0805, symbol R2
- P3: renamed from P8; value DRL_LED -> LED_1
- P4: renamed from P9; value LED_DRV -> LED_2; footprint bebl_v2_pretty:pin_strip_2 -> bebl_v2_pretty:pin_socket_2
- P5: renamed from P10; value LED_DRL -> LED_3; footprint bebl_v2_pretty:pin_strip_2 -> bebl_v2_pretty:pin_socket_2
- P6: renamed from P11; value DRV_LED -> LED_PWR
- P9: renamed from P3; footprint bebl_v2_pretty:pin_strip_2 -> bebl_v2_pretty:pin_socket_2
- renumbered B10 to B7, B14 to B8, B15 to B9, C11 to C10, C13 to C11, C8 to C5, C12 to C6, C10 to C8, L2 to L1, P4 to P7, P12 to P8, R8 to R4, R6 to R5, R7 to R6, U4 to U2, U5 to U3, U3 to U4
Connections:
- wire segments 200 -> 170
Other:
- note added: "6x LED, 2.2V @ 20mA, 5mm, 9000mcd\n(1x Blink, 4x PWM, 1x Digital)\n+ 1x Charge LED"
- note removed: "1x LED 2.2V @ 20mA, 5mm, 9000mcd\n(On Indicator, Day time running light - DRL)"
- note removed: "LED DRIVER"
- moved on the sheet: B8, B9, C10, C11, C5, C6, C7, C8, C9, L1, P3, P4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
