File: kicad/LED_Driver.sch (KiCad schematic (older format))
At the start: 9 parts, among them Q201 MGSF1N03L, Q202 MGSF1N03L, SW201 SWITCH

Commit message: work in progress
Parts:
- R201: footprint bebl_v2_legacy:r_0805 -> (none)
Changed lines of the file:
@@
 F 0 "R201" V 3000 3000 50  0000 C CNN
 F 1 "100R" V 3100 3025 50  0000 C CNN
-F 2 "bebl_v2_legacy:r_0805" H 3100 3025 60  0001 C CNN
+F 2 "" H 3100 3025 60  0001 C CNN
 F 3 "" H 3100 3025 60  0000 C CNN
 	1    3100 3025
