File: kicad/bebl_v2_LED_Driver.sch (KiCad schematic (older format))
At the start: 68 parts, among them P1 ISP, P10 LED_DRL, P11 DRV_LED, P12 CHG_LED, P13 LED_CHG, P2 FTDI, P3 Ext_LiPo, P4 USB-Micro, P8 DRL_LED, P9 LED_DRV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

Commit message: working on transistor based driver for leds
Parts:
- removed Q? (x6): BC847BDW1T1G, SOT-363, symbol BC847BDW1T1G
- added C5: 10uF, bebl_v2_pretty:c_0805, symbol C_NPOL
- added C6: 1uF, bebl_v2_pretty:c_0805, symbol C_NPOL
- added D7: RB520S-30TE61, bebl_v2_pretty:Diode-EMD2, symbol DIODESCH
- added L1: 10uH, bebl_v2_pretty:Inductor_NLCV32, symbol INDUCTOR2
- added R4: 140E, bebl_v2_pretty:r_0805, symbol R
- added R5: 12.4E, bebl_v2_pretty:r_0805, symbol R
- added U2: FAN5346, bebl_v2_pretty:SOT23-6, symbol FAN5346
Connections:
- net labels added: ANOD, CATH, D1A, D1K, DRL, LED_A, LED_K, LED_PWM, SW
- wire segments 168 -> 224
Other:
- moved on the sheet: D1, D2, D3, D4, D5, D6, P10, P11, P8, P9
