File: kicad/bebl_v2.kicad_pcb (KiCad board)
At the start: 2 copper layers, 80 x 44 mm, 72 parts, among them P1 ISP, P10 LED_CHG, P11 LED_1, P12 LED_2, P13 LED_3, P14 LED_PWR, P2 FTDI, P3 LED_1, P4 LED_2, P5 LED_3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

Commit message: making some progress with new layout
Parts:
- D2: value LED_P -> LED_B
- D6: value LED_B -> LED_P
- P11, R10, R11, R7, R8, R9: moved to B.Cu
- moved R12 44.4 mm to (103.2, 65.2)
- moved P13 31.0 mm to (90.0, 75.0)
- moved Q1 30.0 mm to (49.0, 75.0), turned to 180 degrees
- moved R1 28.8 mm to (65.5, 65.2)
- moved R7 25.3 mm to (45.0, 79.8), turned to 180 degrees
- moved R8 22.8 mm to (55.0, 79.8), turned to 180 degrees
- moved R11 22.8 mm to (85.0, 79.8), turned to 180 degrees
- moved Q2 19.7 mm to (69.0, 75.0), turned to 180 degrees
- moved R9 17.0 mm to (65.0, 79.8), turned to 180 degrees
- moved R10 15.5 mm to (75.0, 79.8), turned to 180 degrees
- moved Q3 10.0 mm to (79.0, 75.0), turned to 180 degrees
- moved D1 10.0 mm to (104.0, 75.0)
- moved D7 10.0 mm to (94.0, 75.0)
- moved P10 0.71 mm to (94.0, 79.0), turned to 180 degrees
- moved P14 0.71 mm to (94.0, 71.0), turned to 180 degrees
Connections:
- D2 pad 1: Net-(D6-Pad1) -> Net-(D2-Pad1)
- D2 pad 2: Net-(D6-Pad2) -> Net-(D2-Pad2)
- D3 pad 1: Net-(D5-Pad1) -> Net-(D3-Pad1)
- D3 pad 2: Net-(D5-Pad2) -> Net-(D3-Pad2)
- D5 pad 1: Net-(D3-Pad1) -> Net-(D5-Pad1)
- D5 pad 2: Net-(D3-Pad2) -> Net-(D5-Pad2)
- D6 pad 1: Net-(D2-Pad1) -> Net-(D6-Pad1)
- D6 pad 2: Net-(D2-Pad2) -> Net-(D6-Pad2)
- P14 pad 2: GND -> /LED_brd/GND_LED
- Q1 pad 1: GND -> /LED_brd/GND_LED
- Q1 pad 4: GND -> /LED_brd/GND_LED
- Q2 pad 1: GND -> /LED_brd/GND_LED
- Q2 pad 4: GND -> /LED_brd/GND_LED
- Q3 pad 1: GND -> /LED_brd/GND_LED
- Q3 pad 4: GND -> /LED_brd/GND_LED

Commit message: layout work in progress
Parts:
- P13, R12: moved to B.Cu
- moved P6 65.4 mm to (93.0, 46.0), turned to 180 degrees
- moved P3 35.0 mm to (59.0, 52.5), turned to 0 degrees
- moved P13 31.1 mm to (59.0, 72.5), turned to 0 degrees
- moved P5 29.9 mm to (59.0, 47.5)
- moved P12 22.3 mm to (59.0, 75.0), turned to 180 degrees
- moved P11 22.0 mm to (59.0, 77.5), turned to 0 degrees
- moved P4 22.0 mm to (59.0, 50.0), turned to 0 degrees
- moved R12 14.7 mm to (99.5, 79.5), turned to 180 degrees
- moved C1 11.8 mm to (63.0, 43.5), turned to 270 degrees
- moved Q3 10.0 mm to (89.0, 75.0)
- moved B7 9.04 mm to (39.5, 60.0)
- moved R1 8.79 mm to (74.0, 63.0)
- moved X1 6.80 mm to (58.5, 43.5), turned to 180 degrees
- moved C2 6.67 mm to (54.0, 43.5), turned to 270 degrees
- moved R10 2.51 mm to (72.5, 79.5), turned to 0 degrees
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Routing:
- removed copper zone on F.Cu, net /D1K
- removed copper zone on B.Cu, net GND

Commit message: track layout done. Needs verification
Parts:
- B7: moved to B.Cu
- D2: value LED_B -> LED_P
- D4: value LED_P -> LED_B
- P1, P2: moved to F.Cu
- moved B7 26.8 mm to (64.5, 50.4)
- moved R4 19.8 mm to (64.1, 59.0)
- moved C2 17.1 mm to (58.8, 59.9), turned to 0 degrees
- moved C1 16.4 mm to (63.3, 59.9), turned to 0 degrees
- moved X1 13.4 mm to (61.0, 56.7)
- moved C3 11.2 mm to (71.7, 57.5), turned to 180 degrees
- moved R1 10.7 mm to (83.9, 59.0), turned to 90 degrees
- moved R5 6.24 mm to (84.7, 46.2)
- moved R6 6.20 mm to (84.7, 48.5), turned to 0 degrees
- moved C5 5.40 mm to (87.9, 52.0)
- moved U2 3.20 mm to (81.7, 52.0)
- moved U4 1.55 mm to (82.2, 50.0)
- moved C11 1.52 mm to (87.0, 54.0)
- moved C10 1.50 mm to (87.0, 48.0)
- moved C9 1.50 mm to (87.0, 51.5)
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Connections:
- net /SS renamed /LED_P5
- net Net-(D1-Pad2) renamed /LED_brd/LEDK
- net Net-(P11-Pad1) renamed /LED_brd/LEDP1
- net Net-(P11-Pad2) renamed /LED_brd/LEDP2
- net Net-(P12-Pad1) renamed /LED_brd/LEDD3
- net Net-(P12-Pad2) renamed /LED_brd/LEDP4
- net Net-(P13-Pad1) renamed /LED_brd/LEDP5
- net Net-(P13-Pad2) renamed /LED_brd/LEDB6
- net Net-(P4-Pad2) renamed /LED_P4
- net Net-(P8-Pad2) renamed /LED_K
- P1 pad 3: /SCK -> /LED_B6
- P3 pad 1: /SCK -> /LED_P1
- P3 pad 2: Net-(P3-Pad2) -> /LED_P2
- P4 pad 1: Net-(P4-Pad1) -> /LED_D3
- P5 pad 2: Net-(P5-Pad2) -> /LED_B6
- U1 pad 10: Net-(P4-Pad1) -> /LED_P2
- U1 pad 11: Net-(P5-Pad2) -> /LED_D3
- U1 pad 17: /SCK -> /LED_B6
- U1 pad 9: Net-(P3-Pad2) -> /LED_P1
Routing:
- net GND: track 0.00 -> 255.2 mm, vias 0 -> 4
- net +3.3V: track 0.00 -> 96.5 mm, vias 0 -> 3
- net /LED_brd/GND_LED: track 0.00 -> 90.2 mm, vias 0 -> 1
- net /LED_brd/3V3_LED: track 0.00 -> 79.4 mm
- net /BAT: track 0.00 -> 68.6 mm, vias 0 -> 1
- net /RESET: track 0.00 -> 55.6 mm, vias 0 -> 3
- net /LED_brd/LEDP5: track 0.00 -> 40.7 mm, vias 0 -> 2
- net /VUSB: track 0.00 -> 29.8 mm
- net /LED_brd/LEDB6: track 0.00 -> 29.5 mm
- net /MODE: track 0.00 -> 22.1 mm, vias 0 -> 1
- net /LED_brd/LEDP2: track 0.00 -> 20.7 mm, vias 0 -> 1
- net /LED_brd/LEDK: track 0.00 -> 19.8 mm
- net /LED_brd/LEDD3: track 0.00 -> 18.2 mm
- net /PB7: track 0.00 -> 16.6 mm
- net /SCL: track 0.00 -> 16.2 mm, vias 0 -> 2
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- added copper zone on B.Cu, net /LED_brd/GND_LED
- added copper zone on B.Cu, net GND
