File: kicad/bebl_v2_a.kicad_pcb (KiCad board)
At the start: 2 copper layers, 80 x 44 mm, 72 parts, among them P1 ISP, P10 LED_CHG, P11 LED_1, P12 LED_2, P13 LED_3, P14 LED_PWR, P2 FTDI, P3 LED_1, P4 LED_2, P5 LED_3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

Commit message: work in progress
Parts:
- D4: value LED_D -> LED_B
- D7: value LED_B -> LED_D
- R10, R11, R12, R7, R8, R9: value 22E -> 56E
Routing:
- net /LED_brd/LEDP2: track 21.5 -> 20.7 mm
- net /LED_brd/LEDP1: track 11.9 -> 11.2 mm
