File: kicad/LED_brd.sch (KiCad schematic (older format))
At the start: 21 parts, among them P10 LED_CHG, P11 LED_1, P12 LED_2, P13 LED_3, P14 LED_PWR, Q1 BC847BDW1T1G, Q2 BC847BDW1T1G, Q3 BC847BDW1T1G

Commit message: making some progress with new layout
Connections:
- net GND renamed GND_LED
Changed lines of the file:
@@
 LIBS:power
 LIBS:transistors
+LIBS:bebl_v2-cache
 EELAYER 25 0
 EELAYER END
@@
 $EndComp
 $Comp
-L GND #PWR010
-U 1 1 5481A82F
-P 5925 6400
-F 0 "#PWR010" H 5925 6400 30  0001 C CNN
-F 1 "GND" H 5925 6330 30  0001 C CNN
-F 2 "" H 5925 6400 60  0001 C CNN
-F 3 "" H 5925 6400 60  0001 C CNN
-	1    5925 6400
-	1    0    0    -1
-$EndComp
-$Comp
 L BC847BDW1T1G Q1
 U 1 1 5481A835
@@
 Wire Wire Line
 	3750 5300 3750 6400
-$Comp
-L GND #PWR011
-U 1 1 5481E313
-P 3750 6400
-F 0 "#PWR011" H 3750 6400 30  0001 C CNN
-F 1 "GND" H 3750 6330 30  0001 C CNN
-F 2 "" H 3750 6400 60  0001 C CNN
-F 3 "" H 3750 6400 60  0001 C CNN
-	1    3750 6400
-	1    0    0    -1
-$EndComp
 Wire Wire Line
 	3600 5100 3750 5100
@@
 Wire Wire Line
 	3725 2325 5425 2325
+Wire Wire Line
+	3750 6400 5925 6400
 $EndSCHEMATC

Commit message: track layout done. Needs verification
Parts:
- D2: value LED_B -> LED_P
- D4: value LED_P -> LED_B
Connections:
- net LEDP1: now reaches P11.1 (P1), Q1.2 (B)
- net LEDP2: now reaches P11.2 (PM), Q1.5 (B)
- net LEDD3: now reaches P12.1 (P1), Q2.2 (B)
- net LEDP4: now reaches P12.2 (PM), Q2.5 (B)
- net LEDP5: now reaches P13.1 (P1), Q3.2 (B)
- net LEDB6: now reaches P13.2 (PM), Q3.5 (B)
- net LEDK: now reaches D1.2 (K), P10.2 (PM)
Changed lines of the file:
@@
 P 5650 3350
 F 0 "D2" H 5800 3300 40  0000 C CNN
-F 1 "LED_B" H 5500 3300 40  0000 C CNN
+F 1 "LED_P" H 5500 3300 40  0000 C CNN
 F 2 "bebl_v2_pretty:LED-5MM" H 5650 3350 60  0001 C CNN
 F 3 "" H 5650 3350 60  0000 C CNN
@@
 P 5650 4350
 F 0 "D4" H 5800 4300 40  0000 C CNN
-F 1 "LED_P" H 5475 4300 40  0000 C CNN
+F 1 "LED_B" H 5475 4300 40  0000 C CNN
 F 2 "bebl_v2_pretty:LED-5MM" H 5650 4350 60  0001 C CNN
 F 3 "" H 5650 4350 60  0000 C CNN
@@
 Connection ~ 6525 3350
 Wire Wire Line
-	4100 3550 5000 3550
-Wire Wire Line
-	4200 4050 5000 4050
-Wire Wire Line
-	4200 4550 5000 4550
-Wire Wire Line
-	4100 5050 5000 5050
-Wire Wire Line
-	4000 5550 5000 5550
-Wire Wire Line
-	3900 6050 5000 6050
+	4750 3550 5000 3550
+Wire Wire Line
+	4850 4050 5000 4050
+Wire Wire Line
+	4850 4550 5000 4550
+Wire Wire Line
+	4750 5050 5000 5050
+Wire Wire Line
+	4650 5550 5000 5550
+Wire Wire Line
+	4550 6050 5000 6050
 $Comp
 L DIODE_LED D1
@@
 $EndComp
 Wire Wire Line
-	4100 3550 4100 4050
-Wire Wire Line
-	4100 4050 3600 4050
-Wire Wire Line
-	4200 4050 4200 4250
-Wire Wire Line
-	4200 4250 3600 4250
-Wire Wire Line
-	4200 4550 4200 4400
-Wire Wire Line
-	4200 4400 3600 4400
-Wire Wire Line
-	3600 4600 4100 4600
-Wire Wire Line
-	4100 4600 4100 5050
-Wire Wire Line
-	3600 4750 4000 4750
-Wire Wire Line
-	4000 4750 4000 5550
-Wire Wire Line
-	3600 4950 3900 4950
-Wire Wire Line
-	3900 4950 3900 6050
+	4750 3550 4750 4050
+Wire Wire Line
+	4750 4050 3600 4050
+Wire Wire Line
+	4850 4050 4850 4250
+Wire Wire Line
+	4850 4250 3600 4250
+Wire Wire Line
+	4850 4550 4850 4400
+Wire Wire Line
+	4850 4400 3600 4400
+Wire Wire Line
+	3600 4600 4750 4600
+Wire Wire Line
+	4750 4600 4750 5050
+Wire Wire Line
+	3600 4750 4650 4750
+Wire Wire Line
+	4650 4750 4650 5550
+Wire Wire Line
+	3600 4950 4550 4950
+Wire Wire Line
+	4550 4950 4550 6050
 Wire Wire Line
 	3600 5300 3750 5300
@@
 Wire Wire Line
 	3750 6400 5925 6400
+Text Label 3900 1775 0    39   ~ 0
+LEDK
+Text Label 3950 4050 0    39   ~ 0
+LEDP1
+Text Label 3950 4250 0    39   ~ 0
+LEDP2
+Text Label 3950 4400 0    39   ~ 0
+LEDD3
+Text Label 3950 4600 0    39   ~ 0
+LEDP4
+Text Label 3950 4750 0    39   ~ 0
+LEDP5
+Text Label 3950 4950 0    39   ~ 0
+LEDB6
 $EndSCHEMATC

Commit message: work in progress
Parts:
- D4: value LED_B -> LED_D
- D7: value LED_D -> LED_B
- R10, R11, R12, R7, R8, R9: value 56E -> 22E
Other:
- note added: "LED_B = Blink\nLED_P = PWM\nLED_D = Digital\n\nLED Resistor\n3V3(Supply) - 2V2(LED) - 0.7(transistor) = 0.4V\nRled = 0.4V / 20mA = 20 Ohm\nrounded to 22 Ohm"
- note removed: "LED_B = Blink\nLED_P = PWM\nLED_D = Digital"
Changed lines of the file:
@@
 P 5650 4350
 F 0 "D4" H 5800 4300 40  0000 C CNN
-F 1 "LED_B" H 5475 4300 40  0000 C CNN
+F 1 "LED_D" H 5475 4300 40  0000 C CNN
 F 2 "bebl_v2_pretty:LED-5MM" H 5650 4350 60  0001 C CNN
 F 3 "" H 5650 4350 60  0000 C CNN
@@
 P 5650 5850
 F 0 "D7" H 5800 5800 40  0000 C CNN
-F 1 "LED_D" H 5475 5800 40  0000 C CNN
+F 1 "LED_B" H 5475 5800 40  0000 C CNN
 F 2 "bebl_v2_pretty:LED-5MM" H 5650 5850 60  0001 C CNN
 F 3 "" H 5650 5850 60  0000 C CNN
@@
 P 6200 3350
 F 0 "R7" H 6125 3525 50  0000 C CNN
-F 1 "56E" V 6200 3350 50  0000 C CNN
+F 1 "22E" V 6200 3350 50  0000 C CNN
 F 2 "bebl_v2_pretty:r_0805" H 6200 3350 60  0001 C CNN
 F 3 "" H 6200 3350 60  0000 C CNN
@@
 P 6200 3850
 F 0 "R8" H 6125 4025 50  0000 C CNN
-F 1 "56E" V 6200 3850 50  0000 C CNN
+F 1 "22E" V 6200 3850 50  0000 C CNN
 F 2 "bebl_v2_pretty:r_0805" H 6200 3850 60  0001 C CNN
 F 3 "" H 6200 3850 60  0000 C CNN
@@
 P 6200 4350
 F 0 "R9" H 6125 4525 50  0000 C CNN
-F 1 "56E" V 6200 4350 50  0000 C CNN
+F 1 "22E" V 6200 4350 50  0000 C CNN
 F 2 "bebl_v2_pretty:r_0805" H 6200 4350 60  0001 C CNN
 F 3 "" H 6200 4350 60  0000 C CNN
@@
 P 6200 4850
 F 0 "R10" H 6125 5025 50  0000 C CNN
-F 1 "56E" V 6200 4850 50  0000 C CNN
+F 1 "22E" V 6200 4850 50  0000 C CNN
 F 2 "bebl_v2_pretty:r_0805" H 6200 4850 60  0001 C CNN
 F 3 "" H 6200 4850 60  0000 C CNN
@@
 P 6200 5350
 F 0 "R11" H 6125 5525 50  0000 C CNN
-F 1 "56E" V 6200 5350 50  0000 C CNN
+F 1 "22E" V 6200 5350 50  0000 C CNN
 F 2 "bebl_v2_pretty:r_0805" H 6200 5350 60  0001 C CNN
 F 3 "" H 6200 5350 60  0000 C CNN
@@
 P 6200 5850
 F 0 "R12" H 6125 6025 50  0000 C CNN
-F 1 "56E" V 6200 5850 50  0000 C CNN
+F 1 "22E" V 6200 5850 50  0000 C CNN
 F 2 "bebl_v2_pretty:r_0805" H 6200 5850 60  0001 C CNN
 F 3 "" H 6200 5850 60  0000 C CNN
@@
 Text Label 3750 6250 0    50   ~ 0
 GND_LED
-Text Notes 6975 6400 0    60   ~ 0
-LED_B = Blink\nLED_P = PWM\nLED_D = Digital
+Text Notes 6975 6425 0    59   ~ 0
+LED_B = Blink\nLED_P = PWM\nLED_D = Digital\n\nLED Resistor\n3V3(Supply) - 2V2(LED) - 0.7(transistor) = 0.4V\nRled = 0.4V / 20mA = 20 Ohm\nrounded to 22 Ohm
 Wire Wire Line
 	5875 2325 6525 2325

Commit message: footprint errors corrected, BoM ready, but pending seeed format
Parts:
- Q1, Q2, Q3: footprint bebl_v2_pretty:SOT23-6 -> bebl_v2_pretty:SOT363
Changed lines of the file:
@@
 F 0 "Q1" H 5375 3450 50  0000 C CNN
 F 1 "BC847BDW1T1G" H 5575 3550 40  0000 C CNN
-F 2 "bebl_v2_pretty:SOT23-6" H 5335 3550 30  0001 C CNN
+F 2 "bebl_v2_pretty:SOT363" H 5335 3550 30  0001 C CNN
 F 3 "" H 5175 3550 60  0000 C CNN
 	1    5175 3550
@@
 F 0 "Q1" H 5375 3950 50  0000 C CNN
 F 1 "BC847BDW1T1G" H 5575 4050 40  0000 C CNN
-F 2 "bebl_v2_pretty:SOT23-6" H 5335 4050 30  0001 C CNN
+F 2 "bebl_v2_pretty:SOT363" H 5335 4050 30  0001 C CNN
 F 3 "" H 5175 4050 60  0000 C CNN
 	2    5175 4050
@@
 F 0 "Q2" H 5375 4450 50  0000 C CNN
 F 1 "BC847BDW1T1G" H 5575 4550 40  0000 C CNN
-F 2 "bebl_v2_pretty:SOT23-6" H 5335 4550 30  0001 C CNN
+F 2 "bebl_v2_pretty:SOT363" H 5335 4550 30  0001 C CNN
 F 3 "" H 5175 4550 60  0000 C CNN
 	1    5175 4550
@@
 F 0 "Q2" H 5375 4950 50  0000 C CNN
 F 1 "BC847BDW1T1G" H 5575 5050 40  0000 C CNN
-F 2 "bebl_v2_pretty:SOT23-6" H 5335 5050 30  0001 C CNN
+F 2 "bebl_v2_pretty:SOT363" H 5335 5050 30  0001 C CNN
 F 3 "" H 5175 5050 60  0000 C CNN
 	2    5175 5050
@@
 F 0 "Q3" H 5375 5450 50  0000 C CNN
 F 1 "BC847BDW1T1G" H 5575 5550 40  0000 C CNN
-F 2 "bebl_v2_pretty:SOT23-6" H 5335 5550 30  0001 C CNN
+F 2 "bebl_v2_pretty:SOT363" H 5335 5550 30  0001 C CNN
 F 3 "" H 5175 5550 60  0000 C CNN
 	1    5175 5550
@@
 F 0 "Q3" H 5375 5950 50  0000 C CNN
 F 1 "BC847BDW1T1G" H 5575 6050 40  0000 C CNN
-F 2 "bebl_v2_pretty:SOT23-6" H 5335 6050 30  0001 C CNN
+F 2 "bebl_v2_pretty:SOT363" H 5335 6050 30  0001 C CNN
 F 3 "" H 5175 6050 60  0000 C CNN
 	2    5175 6050
